Commit message: Update urdf and main launch file.

File: openarm_gripette_description/urdf/openarm_right_gripette.urdf (robot description, URDF)
Before this commit: robot openarm_right, 13 links, 12 joints
Joints:
- removed joint r_arm_pitch
- removed joint r_arm_roll
- removed joint r_arm_yaw
- removed joint r_elbow
- removed joint r_wrist_pitch
- removed joint r_wrist_roll
- removed joint r_wrist_roll_mimic
- removed joint r_wrist_yaw
- added joint openarm_joint1: type revolute, parent hfsb6_6060_750_1_step, child dm_j8009p_2_step_1, origin xyz=-0 -0.0925 0.689 rpy=-1.5708 0 -0, axis 0 0 1, limit lower=-2.99999 upper=0.999986 effort=10 velocity=10
- added joint openarm_joint2: type revolute, parent dm_j8009p_2_step_1, child j2_b_2_step, origin xyz=-0.0301 0 -0.06 rpy=-3.14159 -1.5708 0, axis 0 0 1, limit lower=-3.31613 upper=0.174533 effort=10 velocity=10
- added joint openarm_joint3: type revolute, parent j2_b_2_step, child dm_j4340_2_step, origin xyz=-0 -0.06625 0.0301 rpy=-1.5708 -1.5708 0, axis 0 0 1, limit lower=-1.5708 upper=1.5708 effort=10 velocity=10
- added joint openarm_joint4: type revolute, parent dm_j4340_2_step, child dm_j4310_1_2_step, origin xyz=0 -0.03155 -0.15375 rpy=-1.5708 -0 -0, axis 0 0 1, limit lower=-2.44346 upper=0 effort=10 velocity=10
- added joint openarm_joint5: type revolute, parent dm_j4310_1_2_step, child j6_a_3_step, origin xyz=-0 0.0955 0.0315 rpy=1.5708 -0 0, axis 0 0 1, limit lower=-1.5708 upper=1.5708 effort=10 velocity=10
- added joint openarm_joint6: type revolute, parent j6_a_3_step, child j7_e_2_step, origin xyz=0.0172 -0 -0.0455 rpy=-1.5708 -0 1.5708, axis 0 0 1, limit lower=-0.785398 upper=0.785398 effort=10 velocity=10
- added joint openarm_joint6_mimic: type revolute, parent j6_a_3_step, child dm_j4310_1_2_step_2, origin xyz=0.0343 -0 -0.1205 rpy=-1.5708 0 -1.5708, axis 0 0 1, limit lower=-3.141592653589793 upper=3.141592653589793 effort=10 velocity=10, mimic joint=openarm_joint6 multiplier=-1.0
- added joint openarm_joint7: type revolute, parent dm_j4310_1_2_step_2, child gripper_base, origin xyz=0.0205 -0 -0.0343 rpy=0 -1.5708 0, axis 0 0 1, limit lower=-1.5708 upper=1.5708 effort=10 velocity=10

Commit message: Flip axis in urdf.

File: openarm_gripette_description/urdf/openarm_right_gripette.urdf (robot description, URDF)
Before this commit: robot openarm_right, 13 links, 12 joints
Joints:
- joint openarm_joint1: axis 0 0 1 -> 0 0 -1
- joint openarm_joint2: axis 0 0 1 -> 0 0 -1
- joint openarm_joint3: axis 0 0 1 -> 0 0 -1
- joint openarm_joint4: axis 0 0 1 -> 0 0 -1
- joint openarm_joint5: axis 0 0 1 -> 0 0 -1
- joint openarm_joint6: axis 0 0 1 -> 0 0 -1
- joint openarm_joint6_mimic: axis 0 0 1 -> 0 0 -1
- joint openarm_joint7: axis 0 0 1 -> 0 0 -1
